Commit message: Updates focused on getting the simulation working.
- Remove collision definitions from main robot definition file for the chassis as it's only meant for visualization and conflicts with our laser placement in the simulation.
- Adding move_base.launch clone to the igvc_gazebo launch files so that we don't have to either maintain a separate branch or continuously modify the navigation launch file for simulation and real world use.
- Included this new move_base launch file clone in the gazebo launch files so that gmapping and the navigation stack both start up when we run the simulation.

File: src/igvc/igvc_description/robots/igvc.urdf.xacro (robot description, xacro)
@@ -16,9 +16,4 @@
 			</geometry>
 		</visual>
-		<collision>
-			<geometry>
-				<mesh filename="package://igvc_description/meshes/igvc_chassis.DAE" scale="1 1 1" />
-			</geometry>
-		</collision>
 		<inertial>
 			<mass value="${chassis_mass}"/>

Commit message: Got things functioning with new vehicle configuration

File: src/igvc/igvc_description/robots/igvc.urdf.xacro (robot description, xacro)
@@ -13,11 +13,13 @@
 		<visual>
 			<geometry>
-				<mesh filename="package://igvc_description/meshes/igvc_chassis.DAE" scale="1 1 1" />
+				<mesh filename="package://igvc_description/meshes/Metaknight.dae" scale="1 1 1" />
 			</geometry>
+			<origin rpy="0 0 0" xyz="0 0 -.28"/>
 		</visual>
 		<collision>
 			<geometry>
-				<mesh filename="package://igvc_description/meshes/igvc_chassis.DAE" scale="1 1 1" />
+				<mesh filename="package://igvc_description/meshes/Metaknight.dae" scale="1 1 1" />
 			</geometry>
+			<origin rpy="0 0 0" xyz="0 0 -.28"/>
 		</collision>
 		<inertial>
@@ -97,13 +99,13 @@
 	<igvc_caster parent="base_link" lr="left" reflectY="1"/>
 	<!-- Add a camera -->
-	<c920_camera identifier="left" parent="base_link" xPos="-0.6" yPos="0.05" zPos="1.2" roll="0" pitch="0.35" yaw="1.5708"/>
-	<c920_camera identifier="front" parent="base_link" xPos="-0.5" yPos="0.0" zPos="1.2" roll="0" pitch="0.35" yaw="0"/>
-	<c920_camera identifier="right" parent="base_link" xPos="-0.6" yPos="-0.05" zPos="1.2" roll="0" pitch="0.35" yaw="-1.5708"/>
+	<c920_camera identifier="left" parent="base_link" xPos="0.1397" yPos="0.3302" zPos="0.3" roll="0" pitch="0.35" yaw="1.5708"/>
+	<c920_camera identifier="front" parent="base_link" xPos="-0.254" yPos="0.0" zPos="0.863" roll="0" pitch="0.35" yaw="0"/>
+	<c920_camera identifier="right" parent="base_link" xPos="0.1397" yPos="-0.3302" zPos="0.3" roll="0" pitch="0.35" yaw="-1.5708"/>
 	<!-- Add a laser -->
-	<hokuyo_utm30lx parent="base_link" xPos="0.62" yPos="0" zPos="0" roll="0" pitch="0" yaw="0"/>
+	<hokuyo_utm30lx parent="base_link" xPos="0.294" yPos="0" zPos="0.317" roll="0" pitch="0" yaw="0"/>
 	<!-- Add AHRS-8 -->
-	<sparton_ahrs8 parent="base_link" xPos="0.0" yPos="0" zPos="0" roll="0" pitch="0" yaw="0"/>
+	<sparton_ahrs8 parent="base_link" xPos="-0.5842" yPos="0" zPos="0" roll="0" pitch="0" yaw="3.14159"/>
 	<!-- Add GPS -->
-	<minimax_gps parent="base_link" xPos="-0.4" yPos="0" zPos="0.8" roll="0" pitch="0" yaw="0" />
+	<minimax_gps parent="base_link" xPos="-0.381" yPos="0" zPos="1.09" roll="0" pitch="0" yaw="0" />
 	<!-- Set up miscellaneous igvc plugins not related to sensors -->
 	<igvc_gazebo />

File: src/igvc/igvc_description/urdf/igvc_properties.urdf.xacro (robot description, xacro)
@@ -5,7 +5,7 @@
 	<!-- Chassis properties -->
 	<property name="chassis_mass" value="62"/>
-	<property name="chassis_length" value="1.14"/>
-	<property name="chassis_width" value="0.559"/>
-	<property name="chassis_height" value="0.42"/>
+	<property name="chassis_length" value="0.914"/>
+	<property name="chassis_width" value="0.565"/>
+	<property name="chassis_height" value="0.56"/>
 	<property name="chassis_ixx" value="${(chassis_mass*(chassis_length*chassis_length+chassis_height*chassis_height))/12}"/>
 	<property name="chassis_iyy" value="${(chassis_mass*(chassis_height*chassis_height+chassis_width*chassis_width))/12}"/>

Commit message: modified config files for new configuration

File: src/igvc/igvc_description/robots/igvc.urdf.xacro (robot description, xacro)
@@ -62,5 +62,5 @@
 	</link>
 	<joint name="front_fake_laser_joint" type="fixed">
-		<origin xyz="1.0 0 0"/>
+		<origin xyz="1.22 0 0"/>
 		<parent link="base_link"/>
 		<child link="front_fake_laser"/>
@@ -75,5 +75,5 @@
 	</link>
 	<joint name="left_fake_laser_joint" type="fixed">
-		<origin xyz="0.49 0.845 0" rpy="0 0 0.7854"/>
+		<origin xyz="0.53 0.55 0" rpy="0 0 0.7854"/>
 		<parent link="base_link"/>
 		<child link="left_fake_laser"/>
@@ -88,5 +88,5 @@
 	</link>
 	<joint name="right_fake_laser_joint" type="fixed">
-		<origin xyz="0.33 -0.737 0" rpy="0 0 -0.7854"/>
+		<origin xyz="0.46 -0.53 0" rpy="0 0 -0.7854"/>
 		<parent link="base_link"/>
 		<child link="right_fake_laser"/>
@@ -99,7 +99,7 @@
 	<igvc_caster parent="base_link" lr="left" reflectY="1"/>
 	<!-- Add a camera -->
-	<c920_camera identifier="left" parent="base_link" xPos="0.1397" yPos="0.3302" zPos="0.3" roll="0" pitch="0.35" yaw="1.5708"/>
-	<c920_camera identifier="front" parent="base_link" xPos="-0.254" yPos="0.0" zPos="0.863" roll="0" pitch="0.35" yaw="0"/>
-	<c920_camera identifier="right" parent="base_link" xPos="0.1397" yPos="-0.3302" zPos="0.3" roll="0" pitch="0.35" yaw="-1.5708"/>
+	<c920_camera identifier="left" parent="base_link" xPos="0.1397" yPos="0.203" zPos="0.158" roll="0" pitch="0.35" yaw="0.524"/>
+	<c920_camera identifier="front" parent="base_link" xPos="-0.273" yPos="0.0" zPos="0.9" roll="0" pitch="0.35" yaw="0"/>
+	<c920_camera identifier="right" parent="base_link" xPos="0.1397" yPos="-0.203" zPos="0.158" roll="0" pitch="0.35" yaw="-0.524"/>
 	<!-- Add a laser -->
 	<hokuyo_utm30lx parent="base_link" xPos="0.294" yPos="0" zPos="0.317" roll="0" pitch="0" yaw="0"/>
